Commit message: 添加森威的config文件

File: legged_gym/resources/robots/panda7/urdf/panda7_nleg_arm_1008.urdf (robot description, URDF)
Before this commit: robot robot, 26 links, 25 joints
Links:
- link FL_calf: geometry collision box size=0.25 0.04 0.0495; visual mesh filename=../meshes/calf.dae scale=1 1 1
- link FL_hip: geometry visual mesh filename=../meshes/hip.dae scale=1 1 1
- link FL_thigh: geometry visual mesh filename=../meshes/thigh.dae scale=1 1 1
- link FR_calf: geometry collision box size=0.25 0.04 0.0495; visual mesh filename=../meshes/calf.dae scale=1 1 1
- link FR_hip: geometry visual mesh filename=../meshes/hip.dae scale=1 1 1
- link FR_thigh: geometry visual mesh filename=../meshes/thigh_mirror.dae scale=1 1 1
- link RL_calf: geometry collision box size=0.25 0.04 0.0495; visual mesh filename=../meshes/calf.dae scale=1 1 1
- link RL_hip: geometry visual mesh filename=../meshes/hip.dae scale=1 1 1
- link RL_thigh: geometry visual mesh filename=../meshes/thigh.dae scale=1 1 1
- link RR_calf: geometry collision box size=0.25 0.04 0.0495; visual mesh filename=../meshes/calf.dae scale=1 1 1
- link RR_hip: geometry visual mesh filename=../meshes/hip.dae scale=1 1 1
- link RR_thigh: geometry visual mesh filename=../meshes/thigh_mirror.dae scale=1 1 1
- link arm_link0: geometry collision mesh filename=../meshes/link0.dae; visual mesh filename=../meshes/link0.dae
- link arm_link1: geometry collision mesh filename=../meshes/link1.dae; visual mesh filename=../meshes/link1.dae
- link arm_link2: geometry collision mesh filename=../meshes/link2.dae; visual mesh filename=../meshes/link2.dae
- link arm_link3: geometry collision mesh filename=../meshes/link3.dae; visual mesh filename=../meshes/link3.dae
- link arm_link4: geometry collision mesh filename=../meshes/link4.dae; visual mesh filename=../meshes/link4.dae
- link arm_link5: geometry collision mesh filename=../meshes/link5.dae; visual mesh filename=../meshes/link5.dae
- link arm_link6: geometry collision mesh filename=../meshes/link6.dae; visual mesh filename=../meshes/link6.dae
- link base: geometry collision box size=0.99 0.34 0.24; visual mesh filename=../meshes/trunk.dae scale=1 1 1
- link gripper1: geometry collision mesh filename=../meshes/gripper1.dae; visual mesh filename=../meshes/gripper1.dae
- link gripper2: geometry collision mesh filename=../meshes/gripper2.dae; visual mesh filename=../meshes/gripper2.dae

Commit message: 添加panda7，panda7_fixed_arm，panda7_fixed_gripper的配套文件

File: legged_gym/resources/robots/panda7/urdf/panda7_nleg_arm_1008.urdf (robot description, URDF)
Before this commit: robot panda7, 26 links, 25 joints
Links:
- link FL_FOOT: mass 0.0001 -> 0.01
- link FR_FOOT: mass 0.0001 -> 0.01
- link RL_FOOT: mass 0.0001 -> 0.01
- link RR_FOOT: mass 0.0001 -> 0.01
Joints:
- joint arm_joint4: origin xyz=0.251713743388397 -0.0670979052394916 0.049676701967237 rpy=0 0 0 -> xyz=0.251713743388397 -0.0670979052394916 0 rpy=0 0 0

Commit message: 修改跳跃奖励的判断条件，足端和质心位置之间有点差距

File: legged_gym/resources/robots/panda7/urdf/panda7_nleg_arm_1008.urdf (robot description, URDF)
Before this commit: robot panda7, 26 links, 25 joints
Joints:
- joint arm_joint4: origin xyz=0.251713743388397 -0.0670979052394916 0 rpy=0 0 0 -> xyz=0.251713743388397 -0.0670979052394916 0.049677 rpy=0 0 0
