Commit message: 更新太空步轨迹以及trans

File: legged_gym/resources/robots/panda7/urdf/panda7_fixed_arm.urdf (robot description, URDF)
Before this commit: robot robot, 27 links, 26 joints
Joints:
- joint FL_calf_joint: limit lower=-2.53 upper=-0.45 effort=452 velocity=18.8 -> lower=-2.6 upper=-0.45 effort=452 velocity=18.8
- joint FL_thigh_joint: limit lower=-1.78 upper=3.40 effort=180 velocity=21.6 -> lower=-0.78 upper=3.0 effort=180 velocity=21.6
- joint FR_calf_joint: limit lower=-2.53 upper=-0.45 effort=452 velocity=18.8 -> lower=-2.6 upper=-0.45 effort=452 velocity=18.8
- joint FR_thigh_joint: limit lower=-1.78 upper=3.40 effort=180 velocity=21.6 -> lower=-0.78 upper=3.0 effort=180 velocity=21.6
- joint RL_calf_joint: limit lower=-2.53 upper=-0.45 effort=452 velocity=18.8 -> lower=-2.6 upper=-0.45 effort=452 velocity=18.8
- joint RL_thigh_joint: limit lower=-1.30 upper=4.00 effort=180 velocity=21.6 -> lower=-0.78 upper=2.1 effort=180 velocity=21.6
- joint RR_calf_joint: limit lower=-2.53 upper=-0.45 effort=452 velocity=18.8 -> lower=-2.6 upper=-0.45 effort=452 velocity=18.8
- joint RR_thigh_joint: limit lower=-1.30 upper=4.00 effort=180 velocity=21.6 -> lower=-0.78 upper=2.1 effort=180 velocity=21.6

File: legged_gym/resources/robots/panda7/urdf/panda7_fixed_gripper.urdf (robot description, URDF)
Before this commit: robot robot, 27 links, 26 joints
Joints:
- joint FL_calf_joint: limit lower=-2.53 upper=-0.45 effort=452 velocity=18.8 -> lower=-2.6 upper=-0.45 effort=452 velocity=18.8
- joint FL_thigh_joint: limit lower=-1.78 upper=3.40 effort=180 velocity=21.6 -> lower=-0.78 upper=3.0 effort=180 velocity=21.6
- joint FR_calf_joint: limit lower=-2.53 upper=-0.45 effort=452 velocity=18.8 -> lower=-2.6 upper=-0.45 effort=452 velocity=18.8
- joint FR_thigh_joint: limit lower=-1.78 upper=3.40 effort=180 velocity=21.6 -> lower=-0.78 upper=3.0 effort=180 velocity=21.6
- joint RL_calf_joint: limit lower=-2.53 upper=-0.45 effort=452 velocity=18.8 -> lower=-2.6 upper=-0.45 effort=452 velocity=18.8
- joint RL_thigh_joint: limit lower=-1.30 upper=4.00 effort=180 velocity=21.6 -> lower=-0.78 upper=2.1 effort=180 velocity=21.6
- joint RR_calf_joint: limit lower=-2.53 upper=-0.45 effort=452 velocity=18.8 -> lower=-2.6 upper=-0.45 effort=452 velocity=18.8
- joint RR_thigh_joint: limit lower=-1.30 upper=4.00 effort=180 velocity=21.6 -> lower=-0.78 upper=2.1 effort=180 velocity=21.6
- joint arm_joint1: limit lower=-3.14 upper=3.14 effort=100 velocity=100 -> lower=-2.618 upper=2.618 effort=100 velocity=100
- joint arm_joint2: limit lower=-3.6 upper=0.28 effort=100 velocity=100 -> lower=-1.57 upper=0.28 effort=100 velocity=100
- joint arm_joint6: limit lower=-3.14 upper=3.14 effort=100 velocity=100 -> lower=-1.571 upper=1.571 effort=100 velocity=100

File: legged_gym/resources/robots/panda7/urdf/panda7_nleg_arm.urdf (robot description, URDF)
Before this commit: robot robot, 27 links, 26 joints
Joints:
- joint FL_calf_joint: limit lower=-2.53 upper=-0.45 effort=452 velocity=18.8 -> lower=-2.6 upper=-0.45 effort=452 velocity=18.8
- joint FL_thigh_joint: limit lower=-1.78 upper=3.40 effort=180 velocity=21.6 -> lower=-0.78 upper=3.0 effort=180 velocity=21.6
- joint FR_calf_joint: limit lower=-2.53 upper=-0.45 effort=452 velocity=18.8 -> lower=-2.6 upper=-0.45 effort=452 velocity=18.8
- joint FR_thigh_joint: limit lower=-1.78 upper=3.40 effort=180 velocity=21.6 -> lower=-0.78 upper=3.0 effort=180 velocity=21.6
- joint RL_calf_joint: limit lower=-2.53 upper=-0.45 effort=452 velocity=18.8 -> lower=-2.6 upper=-0.45 effort=452 velocity=18.8
- joint RL_thigh_joint: limit lower=-1.30 upper=4.00 effort=180 velocity=21.6 -> lower=-0.78 upper=2.1 effort=180 velocity=21.6
- joint RR_calf_joint: limit lower=-2.53 upper=-0.45 effort=452 velocity=18.8 -> lower=-2.6 upper=-0.45 effort=452 velocity=18.8
- joint RR_thigh_joint: limit lower=-1.30 upper=4.00 effort=180 velocity=21.6 -> lower=-0.78 upper=2.1 effort=180 velocity=21.6
