Commit message: 更改pd参数，添加电机力矩随机化

File: legged_gym/resources/robots/panda7/urdf/panda7_fixed_gripper.urdf (robot description, URDF)
Before this commit: robot robot, 27 links, 26 joints
Joints:
- joint FL_calf_joint: limit lower=-2.6 upper=-0.45 effort=452 velocity=18.8 -> lower=-2.6 upper=-0.45 effort=572 velocity=12.8
- joint FR_calf_joint: limit lower=-2.6 upper=-0.45 effort=452 velocity=18.8 -> lower=-2.6 upper=-0.45 effort=572 velocity=12.8
- joint RL_calf_joint: limit lower=-2.6 upper=-0.45 effort=452 velocity=18.8 -> lower=-2.6 upper=-0.45 effort=572 velocity=12.8
- joint RR_calf_joint: limit lower=-2.6 upper=-0.45 effort=452 velocity=18.8 -> lower=-2.6 upper=-0.45 effort=572 velocity=12.8

Commit message: 添加电机随机化，模型输入60，pd参数150，修改保存模型参数时的迭代次数数据

File: legged_gym/resources/robots/panda7/urdf/panda7_fixed_gripper.urdf (robot description, URDF)
Before this commit: robot robot, 27 links, 26 joints
Links:
- link FL_calf: geometry collision box size=0.25 0.04 0.0495; collision cylinder length=0.05 radius=0.03
- link FR_calf: geometry collision box size=0.25 0.04 0.0495; collision cylinder length=0.05 radius=0.03
- link RL_calf: geometry collision box size=0.25 0.04 0.0495; collision cylinder length=0.05 radius=0.03
- link RR_calf: geometry collision box size=0.25 0.04 0.0495; collision cylinder length=0.05 radius=0.03
