Commit message: swing轨迹最后不是停在正前方，而是从右侧转向左侧

File: legged_gym/resources/robots/panda7_nleg_rm_arm/panda7_nleg_rm_arm_0102.urdf (robot description, URDF)
Before this commit: robot robot, 25 links, 24 joints
Links:
- link RL_calf: geometry collision box size=0.25 0.04 0.0495; collision cylinder length=0.05 radius=0.03
- link RR_calf: geometry collision box size=0.25 0.04 0.0495; collision cylinder length=0.05 radius=0.03
